Commit message: feat: 重新设计为传统四轮小车模型 + 激光默认关闭
模型改造:
- 原模型: 2个大小驱动轮(中) + 2个小滚轮(前/后) 镶嵌在长方体底盘上
- 新模型: 4个等大车轮(半径0.06m) 传统四轮小车布局
  · 后轮驱动(左/右), diff_drive插件控制
  · 前轮随动(左/右), 被动旋转
  · 底盘: 0.50×0.22×0.10 深蓝色车身
  · 轴距0.32m, 轮距0.26m, 离地间隙0.02m

激光传感器:
- always_on: 1 → 0 (初始关闭, 有订阅者时才工作)
- visualize: true → false (默认不显示扫描线)

同步更新 URDF 可视化模型(robot.urdf.xacro)

File: src/robot_description/urdf/robot.urdf.xacro (robot description, xacro)
@@ -1,12 +1,14 @@
 <?xml version="1.0"?>
 <robot xmlns:xacro="http://www.ros.org/wiki/xacro" name="my_robot">
-  <xacro:property name="body_length" value="0.4"/>
-  <xacro:property name="body_width" value="0.3"/>
-  <xacro:property name="body_height" value="0.15"/>
-  <xacro:property name="wheel_radius" value="0.05"/>
-  <xacro:property name="wheel_width" value="0.03"/>
-  <xacro:property name="caster_radius" value="0.03"/>
-  <xacro:macro name="wheel_link" params="name prefix x y z">
-    <link name="${prefix}_${name}_wheel">
+  <xacro:property name="body_length" value="0.50"/>
+  <xacro:property name="body_width" value="0.22"/>
+  <xacro:property name="body_height" value="0.10"/>
+  <xacro:property name="wheel_radius" value="0.06"/>
+  <xacro:property name="wheel_width" value="0.025"/>
+  <xacro:property name="wheelbase" value="0.32"/>   <!-- 前后轴距 -->
+  <xacro:property name="track" value="0.26"/>        <!-- 左右轮距 -->
+  <xacro:property name="clearance" value="0.02"/>    <!-- 底盘离地间隙 -->
+  <xacro:macro name="wheel_link" params="name x y z color">
+    <link name="${name}_link">
       <visual>
         <geometry>
@@ -14,6 +16,6 @@
         </geometry>
         <origin xyz="0 0 0" rpy="${pi/2} 0 0"/>
-        <material name="black">
-          <color rgba="0.2 0.2 0.2 1.0"/>
+        <material name="${name}_mat">
+          <color rgba="${color}"/>
         </material>
       </visual>
@@ -25,39 +27,13 @@
       </collision>
       <inertial>
-        <mass value="0.2"/>
-        <inertia ixx="0.0001" ixy="0.0" ixz="0.0" iyy="0.0001" iyz="0.0" izz="0.0001"/>
+        <mass value="0.15"/>
+        <inertia ixx="0.000143" ixy="0.0" ixz="0.0" iyy="0.00027" iyz="0.0" izz="0.000143"/>
       </inertial>
     </link>
-    <joint name="${prefix}_${name}_wheel_joint" type="continuous">
+    <joint name="${name}_joint" type="continuous">
       <parent link="base_link"/>
-      <child link="${prefix}_${name}_wheel"/>
+      <child link="${name}_link"/>
       <origin xyz="${x} ${y} ${z}" rpy="0 0 0"/>
       <axis xyz="0 1 0"/>
-    </joint>
-  </xacro:macro>
-  <xacro:macro name="caster_link" params="name prefix x y z">
-    <link name="${prefix}_${name}_caster">
-      <visual>
-        <geometry>
-          <sphere radius="${caster_radius}"/>
-        </geometry>
-        <material name="gray">
-          <color rgba="0.5 0.5 0.5 1.0"/>
-        </material>
-      </visual>
-      <collision>
-        <geometry>
-          <sphere radius="${caster_radius}"/>
-        </geometry>
-      </collision>
-      <inertial>
-        <mass value="0.05"/>
-        <inertia ixx="0.00001" ixy="0.0" ixz="0.0" iyy="0.00001" iyz="0.0" izz="0.00001"/>
-      </inertial>
-    </link>
-    <joint name="${prefix}_${name}_caster_joint" type="fixed">
-      <parent link="base_link"/>
-      <child link="${prefix}_${name}_caster"/>
-      <origin xyz="${x} ${y} ${z}" rpy="0 0 0"/>
     </joint>
   </xacro:macro>
@@ -66,5 +42,5 @@
     <parent link="base_footprint"/>
     <child link="base_link"/>
-    <origin xyz="0 0 0.1" rpy="0 0 0"/>
+    <origin xyz="0 0 ${wheel_radius + clearance + body_height/2}" rpy="0 0 0"/>
   </joint>
   <link name="base_link">
@@ -75,5 +51,5 @@
       <origin xyz="0 0 0" rpy="0 0 0"/>
       <material name="blue">
-        <color rgba="0.2 0.4 0.8 1.0"/>
+        <color rgba="0.15 0.2 0.55 1.0"/>
       </material>
     </visual>
@@ -85,31 +61,31 @@
     </collision>
     <inertial>
-      <mass value="2.0"/>
-      <inertia ixx="0.02" ixy="0.0" ixz="0.0" iyy="0.02" iyz="0.0" izz="0.02"/>
+      <mass value="3.0"/>
+      <inertia ixx="0.0146" ixy="0.0" ixz="0.0" iyy="0.065" iyz="0.0" izz="0.0746"/>
     </inertial>
   </link>
-  <xacro:wheel_link name="left" prefix="base" x="0.0" y="${body_width/2 + 0.01}" z="${-body_height/2 + wheel_radius}"/>
-  <xacro:wheel_link name="right" prefix="base" x="0.0" y="${-body_width/2 - 0.01}" z="${-body_height/2 + wheel_radius}"/>
-  <xacro:caster_link name="front" prefix="base" x="${body_length/2 - 0.06}" y="0.0" z="${-body_height/2 + caster_radius - 0.01}"/>
-  <xacro:caster_link name="rear" prefix="base" x="${-body_length/2 + 0.06}" y="0.0" z="${-body_height/2 + caster_radius - 0.01}"/>
+  <xacro:wheel_link name="wheel_left_rear"  x="${-wheelbase/2}" y="${track/2}"  z="${-(body_height/2 + clearance)}" color="0.2 0.2 0.2 1.0"/>
+  <xacro:wheel_link name="wheel_right_rear" x="${-wheelbase/2}" y="${-track/2}" z="${-(body_height/2 + clearance)}" color="0.2 0.2 0.2 1.0"/>
+  <xacro:wheel_link name="wheel_left_front"  x="${wheelbase/2}" y="${track/2}"  z="${-(body_height/2 + clearance)}" color="0.3 0.3 0.3 1.0"/>
+  <xacro:wheel_link name="wheel_right_front" x="${wheelbase/2}" y="${-track/2}" z="${-(body_height/2 + clearance)}" color="0.3 0.3 0.3 1.0"/>
   <link name="lidar_link">
     <visual>
       <geometry>
-        <cylinder radius="0.04" length="0.04"/>
+        <cylinder radius="0.04" length="0.03"/>
       </geometry>
       <origin xyz="0 0 0" rpy="0 0 0"/>
       <material name="red">
-        <color rgba="1.0 0.2 0.2 1.0"/>
+        <color rgba="0.8 0.2 0.2 1.0"/>
       </material>
     </visual>
     <collision>
       <geometry>
-        <cylinder radius="0.04" length="0.04"/>
+        <cylinder radius="0.04" length="0.03"/>
       </geometry>
       <origin xyz="0 0 0" rpy="0 0 0"/>
     </collision>
     <inertial>
-      <mass value="0.1"/>
-      <inertia ixx="0.0001" ixy="0.0" ixz="0.0" iyy="0.0001" iyz="0.0" izz="0.0001"/>
+      <mass value="0.01"/>
+      <inertia ixx="0.000001" ixy="0.0" ixz="0.0" iyy="0.000001" iyz="0.0" izz="0.000001"/>
     </inertial>
   </link>
@@ -117,5 +93,31 @@
     <parent link="base_link"/>
     <child link="lidar_link"/>
-    <origin xyz="0 0 ${body_height/2 + 0.04}" rpy="0 0 0"/>
+    <origin xyz="0 0 ${body_height/2 + 0.015}" rpy="0 0 0"/>
+  </joint>
+  <link name="camera_link">
+    <visual>
+      <geometry>
+        <box size="0.02 0.04 0.02"/>
+      </geometry>
+      <origin xyz="0 0 0" rpy="0 0 0"/>
+      <material name="green">
+        <color rgba="0 0.7 0 1.0"/>
+      </material>
+    </visual>
+    <collision>
+      <geometry>
+        <box size="0.02 0.04 0.02"/>
+      </geometry>
+      <origin xyz="0 0 0" rpy="0 0 0"/>
+    </collision>
+    <inertial>
+      <mass value="0.005"/>
+      <inertia ixx="0.000001" ixy="0.0" ixz="0.0" iyy="0.000001" iyz="0.0" izz="0.000001"/>
+    </inertial>
+  </link>
+  <joint name="camera_joint" type="fixed">
+    <parent link="base_link"/>
+    <child link="camera_link"/>
+    <origin xyz="${body_length/2 - 0.02} 0 ${body_height/2 - 0.01}" rpy="0 0 0"/>
   </joint>
 </robot>

Commit message: refactor: 替换为官方 TurtleBot3 Waffle 机器人模型
彻底删除旧的自定义机器人模型，改用官方 TurtleBot3 Waffle:

模型来源: ROBOTIS 官方 turtlebot3_gazebo / turtlebot3_description 包
规格: 差速驱动 | 轮径0.066m/轮距0.287m | LDS-01激光雷达 | IMU | RealSense R200相机

修改文件清单 (11个文件):

1. 删除: src/robot_proj/models/custom_robot/ (旧自定义模型)
2. 新增: models/turtlebot3_waffle/ (TurtleBot3 Waffle SDF)
   - LiDAR always_on=0, visualize=false (默认关闭, 订阅时自动开启)
3. classroom_sim.launch.py → 指向新模型路径
4. MainWindow.cpp → 更新SDF加载路径
5. 地面接触参数: classroom.world 新增 kp=1e5/kd=1 接触约束
   (配合TB3车轮 mu≈∞ 摩擦, 确保零滑移/零弹跳)
6. robot.urdf.xacro → 重写为 TurtleBot3 Waffle 完整URDF
7. rviz.launch.py → 使用 turtlebot3_description 官方URDF
8. package.xml → 新增依赖 turtlebot3_gazebo / turtlebot3_description
9. README.md → 更新模型说明、抓地力参数、话题对照表

ROS话题(命名空间 robot_01):
  /robot_01/cmd_vel | /robot_01/odom | /robot_01/scan
  /robot_01/imu | /robot_01/camera/image_raw | /robot_01/joint_states

File: src/robot_description/urdf/robot.urdf.xacro (robot description, xacro)
@@ -1,123 +1,174 @@
 <?xml version="1.0"?>
-<robot xmlns:xacro="http://www.ros.org/wiki/xacro" name="my_robot">
-  <xacro:property name="body_length" value="0.50"/>
-  <xacro:property name="body_width" value="0.22"/>
-  <xacro:property name="body_height" value="0.10"/>
-  <xacro:property name="wheel_radius" value="0.06"/>
-  <xacro:property name="wheel_width" value="0.025"/>
-  <xacro:property name="wheelbase" value="0.32"/>   <!-- 前后轴距 -->
-  <xacro:property name="track" value="0.26"/>        <!-- 左右轮距 -->
-  <xacro:property name="clearance" value="0.02"/>    <!-- 底盘离地间隙 -->
-  <xacro:macro name="wheel_link" params="name x y z color">
-    <link name="${name}_link">
-      <visual>
-        <geometry>
-          <cylinder radius="${wheel_radius}" length="${wheel_width}"/>
-        </geometry>
-        <origin xyz="0 0 0" rpy="${pi/2} 0 0"/>
-        <material name="${name}_mat">
-          <color rgba="${color}"/>
-        </material>
-      </visual>
-      <collision>
-        <geometry>
-          <cylinder radius="${wheel_radius}" length="${wheel_width}"/>
-        </geometry>
-        <origin xyz="0 0 0" rpy="${pi/2} 0 0"/>
-      </collision>
-      <inertial>
-        <mass value="0.15"/>
-        <inertia ixx="0.000143" ixy="0.0" ixz="0.0" iyy="0.00027" iyz="0.0" izz="0.000143"/>
-      </inertial>
-    </link>
-    <joint name="${name}_joint" type="continuous">
-      <parent link="base_link"/>
-      <child link="${name}_link"/>
-      <origin xyz="${x} ${y} ${z}" rpy="0 0 0"/>
-      <axis xyz="0 1 0"/>
-    </joint>
-  </xacro:macro>
-  <link name="base_footprint"/>
-  <joint name="base_joint" type="fixed">
-    <parent link="base_footprint"/>
-    <child link="base_link"/>
-    <origin xyz="0 0 ${wheel_radius + clearance + body_height/2}" rpy="0 0 0"/>
+<!-- TurtleBot3 Waffle 机器人描述文件（RViz 可视化用） -->
+<!-- 基于官方 turtlebot3_description 包 -->
+<robot xmlns:xacro="http://www.ros.org/wiki/xacro" name="turtlebot3_waffle">
+  <xacro:arg name="namespace" default=""/>
+  <xacro:property name="namespace" value="$(arg namespace)"/>
+  <material name="black"><color rgba="0.0 0.0 0.0 1.0"/></material>
+  <material name="dark"><color rgba="0.3 0.3 0.3 1.0"/></material>
+  <material name="light_black"><color rgba="0.4 0.4 0.4 1.0"/></material>
+  <material name="blue"><color rgba="0.0 0.0 0.8 1.0"/></material>
+  <material name="green"><color rgba="0.0 0.8 0.0 1.0"/></material>
+  <material name="red"><color rgba="0.8 0.0 0.0 1.0"/></material>
+  <link name="${namespace}base_footprint"/>
+  <joint name="${namespace}base_joint" type="fixed">
+    <parent link="${namespace}base_footprint"/>
+    <child link="${namespace}base_link"/>
+    <origin xyz="0 0 0.010" rpy="0 0 0"/>
   </joint>
-  <link name="base_link">
+  <link name="${namespace}base_link">
     <visual>
+      <origin xyz="-0.064 0 0" rpy="0 0 0"/>
       <geometry>
-        <box size="${body_length} ${body_width} ${body_height}"/>
+        <mesh filename="package://turtlebot3_description/meshes/bases/waffle_base.stl" scale="0.001 0.001 0.001"/>
       </geometry>
-      <origin xyz="0 0 0" rpy="0 0 0"/>
-      <material name="blue">
-        <color rgba="0.15 0.2 0.55 1.0"/>
-      </material>
+      <material name="light_black"/>
     </visual>
     <collision>
-      <geometry>
-        <box size="${body_length} ${body_width} ${body_height}"/>
-      </geometry>
-      <origin xyz="0 0 0" rpy="0 0 0"/>
+      <origin xyz="-0.064 0 0.047" rpy="0 0 0"/>
+      <geometry><box size="0.266 0.266 0.094"/></geometry>
     </collision>
     <inertial>
-      <mass value="3.0"/>
-      <inertia ixx="0.0146" ixy="0.0" ixz="0.0" iyy="0.065" iyz="0.0" izz="0.0746"/>
+      <mass value="1.3729"/>
+      <inertia ixx="0.0087" ixy="-4.76e-5" ixz="1.12e-4"
+               iyy="0.00862" iyz="-3.54e-6"
+               izz="0.01461"/>
     </inertial>
   </link>
-  <xacro:wheel_link name="wheel_left_rear"  x="${-wheelbase/2}" y="${track/2}"  z="${-(body_height/2 + clearance)}" color="0.2 0.2 0.2 1.0"/>
-  <xacro:wheel_link name="wheel_right_rear" x="${-wheelbase/2}" y="${-track/2}" z="${-(body_height/2 + clearance)}" color="0.2 0.2 0.2 1.0"/>
-  <xacro:wheel_link name="wheel_left_front"  x="${wheelbase/2}" y="${track/2}"  z="${-(body_height/2 + clearance)}" color="0.3 0.3 0.3 1.0"/>
-  <xacro:wheel_link name="wheel_right_front" x="${wheelbase/2}" y="${-track/2}" z="${-(body_height/2 + clearance)}" color="0.3 0.3 0.3 1.0"/>
-  <link name="lidar_link">
+  <!-- 左驱动轮 -->
+  <joint name="${namespace}wheel_left_joint" type="continuous">
+    <parent link="${namespace}base_link"/>
+    <child link="${namespace}wheel_left_link"/>
+    <origin xyz="0.0 0.144 0.023" rpy="-1.57 0 0"/>
+    <axis xyz="0 0 1"/>
+  </joint>
+  <link name="${namespace}wheel_left_link">
     <visual>
+      <origin xyz="0 0 0" rpy="1.57 0 0"/>
       <geometry>
-        <cylinder radius="0.04" length="0.03"/>
+        <mesh filename="package://turtlebot3_description/meshes/wheels/left_tire.stl" scale="0.001 0.001 0.001"/>
       </geometry>
-      <origin xyz="0 0 0" rpy="0 0 0"/>
-      <material name="red">
-        <color rgba="0.8 0.2 0.2 1.0"/>
-      </material>
+      <material name="dark"/>
     </visual>
     <collision>
-      <geometry>
-        <cylinder radius="0.04" length="0.03"/>
-      </geometry>
-      <origin xyz="0 0 0" rpy="0 0 0"/>
+      <geometry><cylinder length="0.018" radius="0.033"/></geometry>
     </collision>
     <inertial>
-      <mass value="0.01"/>
-      <inertia ixx="0.000001" ixy="0.0" ixz="0.0" iyy="0.000001" iyz="0.0" izz="0.000001"/>
+      <mass value="0.0285"/>
+      <inertia ixx="1.12e-5" ixy="0" ixz="0" iyy="1.12e-5" iyz="0" izz="2.07e-5"/>
     </inertial>
   </link>
-  <joint name="lidar_joint" type="fixed">
-    <parent link="base_link"/>
-    <child link="lidar_link"/>
-    <origin xyz="0 0 ${body_height/2 + 0.015}" rpy="0 0 0"/>
+  <!-- 右驱动轮 -->
+  <joint name="${namespace}wheel_right_joint" type="continuous">
+    <parent link="${namespace}base_link"/>
+    <child link="${namespace}wheel_right_link"/>
+    <origin xyz="0.0 -0.144 0.023" rpy="-1.57 0 0"/>
+    <axis xyz="0 0 1"/>
   </joint>
-  <link name="camera_link">
+  <link name="${namespace}wheel_right_link">
     <visual>
+      <origin xyz="0 0 0" rpy="1.57 0 0"/>
       <geometry>
-        <box size="0.02 0.04 0.02"/>
+        <mesh filename="package://turtlebot3_description/meshes/wheels/right_tire.stl" scale="0.001 0.001 0.001"/>
       </geometry>
-      <origin xyz="0 0 0" rpy="0 0 0"/>
-      <material name="green">
-        <color rgba="0 0.7 0 1.0"/>
-      </material>
+      <material name="dark"/>
     </visual>
     <collision>
-      <geometry>
-        <box size="0.02 0.04 0.02"/>
-      </geometry>
-      <origin xyz="0 0 0" rpy="0 0 0"/>
+      <geometry><cylinder length="0.018" radius="0.033"/></geometry>
+    </collision>
+    <inertial>
+      <mass value="0.0285"/>
+      <inertia ixx="1.12e-5" ixy="0" ixz="0" iyy="1.12e-5" iyz="0" izz="2.07e-5"/>
+    </inertial>
+  </link>
+  <!-- 后万向轮 -->
+  <link name="${namespace}caster_back_right_link">
+    <collision>
+      <origin xyz="0 0.001 0" rpy="0 0 0"/>
+      <geometry><box size="0.030 0.009 0.020"/></geometry>
     </collision>
     <inertial>
       <mass value="0.005"/>
-      <inertia ixx="0.000001" ixy="0.0" ixz="0.0" iyy="0.000001" iyz="0.0" izz="0.000001"/>
+      <inertia ixx="0.001" ixy="0" ixz="0" iyy="0.001" iyz="0" izz="0.001"/>
     </inertial>
   </link>
-  <joint name="camera_joint" type="fixed">
-    <parent link="base_link"/>
-    <child link="camera_link"/>
-    <origin xyz="${body_length/2 - 0.02} 0 ${body_height/2 - 0.01}" rpy="0 0 0"/>
+  <joint name="${namespace}caster_back_right_joint" type="fixed">
+    <parent link="${namespace}base_link"/>
+    <child link="${namespace}caster_back_right_link"/>
+    <origin xyz="-0.177 -0.064 -0.004" rpy="-1.57 0 0"/>
+  </joint>
+  <link name="${namespace}caster_back_left_link">
+    <collision>
+      <origin xyz="0 0.001 0" rpy="0 0 0"/>
+      <geometry><box size="0.030 0.009 0.020"/></geometry>
+    </collision>
+    <inertial>
+      <mass value="0.005"/>
+      <inertia ixx="0.001" ixy="0" ixz="0" iyy="0.001" iyz="0" izz="0.001"/>
+    </inertial>
+  </link>
+  <joint name="${namespace}caster_back_left_joint" type="fixed">
+    <parent link="${namespace}base_link"/>
+    <child link="${namespace}caster_back_left_link"/>
+    <origin xyz="-0.177 0.064 -0.004" rpy="-1.57 0 0"/>
+  </joint>
+  <!-- IMU -->
+  <link name="${namespace}imu_link"/>
+  <joint name="${namespace}imu_joint" type="fixed">
+    <parent link="${namespace}base_link"/>
+    <child link="${namespace}imu_link"/>
+    <origin xyz="0 0 0.068" rpy="0 0 0"/>
+  </joint>
+  <!-- LiDAR -->
+  <link name="${namespace}base_scan">
+    <visual>
+      <geometry>
+        <mesh filename="package://turtlebot3_description/meshes/sensors/lds.stl" scale="0.001 0.001 0.001"/>
+      </geometry>
+      <material name="dark"/>
+    </visual>
+    <collision>
+      <origin xyz="0.015 0 -0.0065" rpy="0 0 0"/>
+      <geometry><cylinder length="0.0315" radius="0.055"/></geometry>
+    </collision>
+    <inertial>
+      <mass value="0.114"/>
+      <inertia ixx="0.001" ixy="0" ixz="0" iyy="0.001" iyz="0" izz="0.001"/>
+    </inertial>
+  </link>
+  <joint name="${namespace}scan_joint" type="fixed">
+    <parent link="${namespace}base_link"/>
+    <child link="${namespace}base_scan"/>
+    <origin xyz="-0.064 0 0.122" rpy="0 0 0"/>
+  </joint>
+  <!-- 摄像头 -->
+  <link name="${namespace}camera_link">
+    <visual>
+      <origin xyz="0 0 0" rpy="1.57 0 1.57"/>
+      <geometry>
+        <mesh filename="package://turtlebot3_description/meshes/sensors/r200.dae"/>
+      </geometry>
+    </visual>
+    <collision>
+      <origin xyz="0.003 0.065 0.007" rpy="0 0 0"/>
+      <geometry><box size="0.012 0.132 0.020"/></geometry>
+    </collision>
+  </link>
+  <joint name="${namespace}camera_joint" type="fixed">
+    <parent link="${namespace}base_link"/>
+    <child link="${namespace}camera_link"/>
+    <origin xyz="0.064 -0.065 0.094" rpy="0 0 0"/>
+  </joint>
+  <link name="${namespace}camera_rgb_frame"/>
+  <joint name="${namespace}camera_rgb_joint" type="fixed">
+    <parent link="${namespace}camera_link"/>
+    <child link="${namespace}camera_rgb_frame"/>
+    <origin xyz="0.005 0.018 0.013" rpy="0 0 0"/>
+  </joint>
+  <link name="${namespace}camera_rgb_optical_frame"/>
+  <joint name="${namespace}camera_rgb_optical_joint" type="fixed">
+    <parent link="${namespace}camera_rgb_frame"/>
+    <child link="${namespace}camera_rgb_optical_frame"/>
+    <origin xyz="0 0 0" rpy="-1.57 0 -1.57"/>
   </joint>
 </robot>

Commit message: fix: 匀速控制 + 相机翻转 + 后置摄像头
1. 速度不均匀修复 (RobotController):
   原: 按前进键只发布1次cmd_vel → diff_drive约0.5s看门狗超时自动停止
   → 表现为'快一段→慢下来→再按再快-慢'
   新: 添加50ms定时器, 按键按住期间持续发布cmd_vel (20Hz)
   松开按键→停止定时器+发布零速, 配合accel=10.0实现~1.5s制动

2. 相机上下颠倒修复 (RosCameraWidget):
   移除 img.mirrored(false, true) 的错误垂直翻转
   Gazebo相机数据row0=顶部, QImage row0=顶部, 无需翻转

3. 后置摄像头 (TB3模型尾部):
   新增 camera_rear_link (位置-0.15,0,0.08, yaw=180°)
   640x480 RGB, 发布到 /robot_01/rear_camera/image_raw
   backCamWidget → 后方视角 / frontCamWidget → 前方视角
   同步更新 URDF 可视化模型

File: src/robot_description/urdf/robot.urdf.xacro (robot description, xacro)
@@ -172,3 +172,14 @@
     <origin xyz="0 0 0" rpy="-1.57 0 -1.57"/>
   </joint>
+  <!-- 后置摄像头（尾部朝后） -->
+  <link name="${namespace}camera_rear_link">
+    <visual>
+      <geometry><box size="0.015 0.03 0.015"/></geometry>
+      <material name="blue"/>
+    </visual>
+    <inertial>
+      <mass value="0.001"/>
+      <inertia ixx="1e-6" ixy="0" ixz="0" iyy="1e-6" iyz="0" izz="1e-6"/>
+    </inertial>
+  </link>
 </robot>
